File: FrameGuard.kicad_pcb (KiCad board)
At the start: 4 copper layers, 70.9 x 71.2 mm, 43 parts, among them J1 USB_C_Receptacle_USB2.0_16P, J5 Conn_01x06_Socket, J6 Conn_01x04_Socket, Q11 RTQ045N03HZGTR, SW1 SW_Push, SW2 SW_Push, U1 ESP32-S3-WROOM-1, U2 TPD4E001DBVR, U3 TPS22917DBV, U4 TLV61225DCKR

Commit message: organization
Parts:
- B1: footprint Batt:1090_KEY -> FrameGuard:BATTERY-1090_KEY
- LS1: footprint Buzzer:XDCR_AT-1127-ST-2-R -> FrameGuard:BUZZER-XDCR_AT-1127-ST-2-R
- S1: footprint Switch:SW_SLW-12689-4A-N-D -> FrameGuard:SWITCH-SW_SLW-12689-4A-N-D
- moved R4 0.43 mm to (157.1, 50.2)
- renumbered GND to TP1, 3V to TP2, 3V3 to TP3

Commit message: small fix
Parts:
- renumbered TP2 to 3V, TP3 to 3V3, TP1 to GND
