File: FrameGuard.kicad_pcb (KiCad board)
At the start: 4 copper layers, 70.9 x 71.2 mm, 43 parts, among them J1 USB_C_Receptacle_USB2.0_16P, J5 Conn_01x06_Socket, J6 Conn_01x04_Socket, Q11 RTQ045N03HZGTR, SW1 SW_Push, SW2 SW_Push, U1 ESP32-S3-WROOM-1, U2 TPD4E001DBVR, U3 TPS22917DBV, U4 TLV61225DCKR

Commit message: changed alarm
Parts:
- LS1: value AT-1127-ST-2-R -> CMI-1295IC-0385T; footprint FrameGuard:BUZZER-XDCR_AT-1127-ST-2-R -> FrameGuard:BUZZER-CUI_CMI-1295IC-0385T
- moved LS1 0.40 mm to (104.0, 49.6), turned to 90 degrees
