File: FrameGuard.kicad_sch (KiCad schematic)
At the start: 43 parts, among them J1 USB_C_Receptacle_USB2.0_16P, J5 Conn_01x06_Socket, J6 Conn_01x04_Socket, Q11 RTQ045N03HZGTR, SW1 SW_Push, SW2 SW_Push, U1 ESP32-S3-WROOM-1, U2 TPD4E001DBVR, U3 TPS22917DBV, U4 TLV61225DCKR

Commit message: organization
Parts:
- B1: footprint Batt:1090_KEY -> FrameGuard:BATTERY-1090_KEY
- LS1: footprint Buzzer:XDCR_AT-1127-ST-2-R -> FrameGuard:BUZZER-XDCR_AT-1127-ST-2-R
- S1: footprint Switch:SW_SLW-12689-4A-N-D -> FrameGuard:SWITCH-SW_SLW-12689-4A-N-D
Changed lines of the file:
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@@
 			)
 		)
-		(property "Footprint" "Buzzer:XDCR_AT-1127-ST-2-R"
+		(property "Footprint" "FrameGuard:BUZZER-XDCR_AT-1127-ST-2-R"
 			(at 81.28 29.21 0)
 			(hide yes)
@@
 			)
 		)
-		(property "Footprint" "Batt:1090_KEY"
+		(property "Footprint" "FrameGuard:BATTERY-1090_KEY"
 			(at 38.1 90.17 0)
 			(hide yes)
@@
 			)
 		)
-		(property "Footprint" "Switch:SW_SLW-12689-4A-N-D"
+		(property "Footprint" "FrameGuard:SWITCH-SW_SLW-12689-4A-N-D"
 			(at 138.43 99.06 0)
 			(hide yes)

Commit message: changed alarm
Parts:
- removed LS1: AT-1127-ST-2-R, FrameGuard:BUZZER-XDCR_AT-1127-ST-2-R, symbol FrameGuardBuzzer:AT-1127-ST-2-R
- added LS1: CMI-1295IC-0385T, FrameGuard:BUZZER-CUI_CMI-1295IC-0385T, symbol FrameGuard:CMI-1295IC-0385T
Connections:
- net +3V3: now also LS1.P
- net at Q11.1 (D), Q11.2 (D), Q11.5 (D)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: now also LS1.N
Changed lines of the file:
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@@
-	)
-	(symbol
-		(lib_id "FrameGuardBuzzer:AT-1127-ST-2-R")
-		(at 81.28 29.21 0)
-		(unit 1)
-		(body_style 1)
-		(exclude_from_sim no)
-		(in_bom yes)
-		(on_board yes)
-		(in_pos_files yes)
-		(dnp no)
-		(fields_autoplaced yes)
-		(property "Reference" "LS1"
-			(at 85.09 28.0842 0)
-			(show_name no)
-			(do_not_autoplace no)
-			(effects
-				(font
-					(size 1.27 1.27)
-				)
-				(justify left)
-			)
-		)
-		(property "Value" "AT-1127-ST-2-R"
-			(at 85.09 30.6242 0)
-			(show_name no)
-			(do_not_autoplace no)
-			(effects
-				(font
-					(size 1.27 1.27)
-				)
-				(justify left)
-			)
-		)
-		(property "Footprint" "FrameGuard:BUZZER-XDCR_AT-1127-ST-2-R"
-			(at 81.28 29.21 0)
-			(hide yes)
-			(show_name no)
-			(do_not_autoplace no)
-			(effects
-				(font
-					(size 1.27 1.27)
-				)
-				(justify bottom)
-			)
-		)
-		(property "Datasheet" "https://www.digikey.com/en/products/detail/pui-audio-inc/AT-1127-ST-2-R/5011397"
-			(at 81.28 29.21 0)
-			(hide yes)
-			(show_name no)
-			(do_not_autoplace no)
-			(effects
-				(font
-					(size 1.27 1.27)
-				)
-			)
-		)
-		(property "Description" ""
-			(at 81.28 29.21 0)
-			(hide yes)
-			(show_name no)
-			(do_not_autoplace no)
-			(effects
-				(font
-					(size 1.27 1.27)
-				)
-			)
-		)
-		(property "PARTREV" "C"
-			(at 81.28 29.21 0)
-			(hide yes)
-			(show_name no)
-			(do_not_autoplace no)
-			(effects
-				(font
-					(size 1.27 1.27)
-				)
-				(justify bottom)
-			)
-		)
-		(property "STANDARD" "Manufacturer Recommendations"
-			(at 81.28 29.21 0)
-			(hide yes)
-			(show_name no)
-			(do_not_autoplace no)
-			(effects
-				(font
-					(size 1.27 1.27)
-				)
-				(justify bottom)
-			)
-		)
-		(property "MAXIMUM_PACKAGE_HEIGHT" "4.2 mm"
-			(at 81.28 29.21 0)
-			(hide yes)
-			(show_name no)
-			(do_not_autoplace no)
-			(effects
-				(font
-					(size 1.27 1.27)
-				)
-				(justify bottom)
-			)
-		)
-		(property "MANUFACTURER" "PUI Audio"
-			(at 81.28 29.21 0)
-			(hide yes)
-			(show_name no)
-			(do_not_autoplace no)
-			(effects
-				(font
-					(size 1.27 1.27)
-				)
-				(justify bottom)
-			)
-		)
-		(pin "P"
-		)
-		(pin "N"
-		)
-		(instances
-			(project "FrameGuard"
-				(path "/677acfd4-1292-4313-917f-731b091b5165"
-					(reference "LS1")
-					(unit 1)
-				)
-			)
-		)
 	)
 	(symbol
@@
 					(unit 1)
 				)
+			)
+		)
+	)
+	(symbol
+		(lib_id "FrameGuard:CMI-1295IC-0385T")
+		(at 81.28 29.21 0)
+		(unit 1)
+		(body_style 1)
+		(exclude_from_sim no)
+		(in_bom yes)
+		(on_board yes)
+		(in_pos_files yes)
+		(dnp no)
+		(fields_autoplaced yes)
+		(property "Reference" "LS1"
+			(at 85.09 27.9399 0)
+			(show_name no)
+			(do_not_autoplace no)
+			(effects
+				(font
+					(size 1.27 1.27)
+				)
+				(justify left)
+			)
+		)
+		(property "Value" "CMI-1295IC-0385T"
+			(at 85.09 30.4799 0)
+			(show_name no)
+			(do_not_autoplace no)
+			(effects
+				(font
+					(size 1.27 1.27)
+				)
+				(justify left)
+			)
+		)
+		(property "Footprint" "FrameGuard:BUZZER-CUI_CMI-1295IC-0385T"
+			(at 81.28 29.21 0)
+			(hide yes)
+			(show_name no)
+			(do_not_autoplace no)
+			(effects
+				(font
+					(size 1.27 1.27)
+				)
+				(justify bottom)
+			)
+		)
+		(property "Datasheet" ""
+			(at 81.28 29.21 0)
+			(hide yes)
+			(show_name no)
+			(do_not_autoplace no)
+			(effects
+				(font
+					(size 1.27 1.27)
+				)
+			)
+		)
+		(property "Description" ""
+			(at 81.28 29.21 0)
+			(hide yes)
+			(show_name no)
+			(do_not_autoplace no)
+			(effects
+				(font
+					(size 1.27 1.27)
+				)
+			)
+		)
+		(property "PARTREV" "1.0"
+			(at 81.28 29.21 0)
+			(hide yes)
+			(show_name no)
+			(do_not_autoplace no)
+			(effects
+				(font
+					(size 1.27 1.27)
+				)
+				(justify bottom)
+			)
+		)
+		(property "STANDARD" "Manufacturer Recommendations"
+			(at 81.28 29.21 0)
+			(hide yes)
+			(show_name no)
+			(do_not_autoplace no)
+			(effects
+				(font
+					(size 1.27 1.27)
+				)
+				(justify bottom)
+			)
+		)
+		(property "MAXIMUM_PACKAGE_HEIGHT" "9.7mm"
+			(at 81.28 29.21 0)
+			(hide yes)
+			(show_name no)
+			(do_not_autoplace no)
+			(effects
+				(font
+					(size 1.27 1.27)
+				)
+				(justify bottom)
+			)
+		)
+		(property "MANUFACTURER" "CUI Inc."
+			(at 81.28 29.21 0)
+			(hide yes)
+			(show_name no)
+			(do_not_autoplace no)
+			(effects
+				(font
+					(size 1.27 1.27)
+				)
+				(justify bottom)
+			)
+		)
+		(pin "N"
+		)
+		(pin "P"
+		)
+		(instances
+			(project "FrameGuard"
+				(path "/677acfd4-1292-4313-917f-731b091b5165"
+					(reference "LS1")
+					(unit 1)
+				)
